File: prototrial/circuit/esplcd/esplcd.kicad_pcb (KiCad board)
At the start: 2 copper layers, 2 parts, among them U1 ESP-12E

Commit message: esp lcd draft
Parts:
- added J-PROG1: Conn_01x06_Male, Connector_PinHeader_2.54mm:PinHeader_1x06_P2.54mm_Vertical, F.Cu at (265.4, 31.8)
- added R-PROG1: 10K, Resistor_SMD:R_0805_2012Metric_Pad1.20x1.40mm_HandSolder, F.Cu at (258.0, 23.8)
- added R-PROG2: 10K, Resistor_SMD:R_0805_2012Metric_Pad1.20x1.40mm_HandSolder, F.Cu at (262.7, 23.8)
- added R-PROG3: 10K, Resistor_SMD:R_0805_2012Metric_Pad1.20x1.40mm_HandSolder, F.Cu at (267.5, 23.8)
- added R-PROG4: 10K, Resistor_SMD:R_0805_2012Metric_Pad1.20x1.40mm_HandSolder, F.Cu at (255.4, 30.6)
- added R-PROG5: 10K, Resistor_SMD:R_0805_2012Metric_Pad1.20x1.40mm_HandSolder, F.Cu at (260.2, 30.6)
- moved U1 4.97 mm to (243.9, 39.7)

Commit message: paging jalan
Parts:
- added J-STM32UART1: Conn_01x03_Male, Connector_Molex:Molex_KK-254_AE-6410-03A_1x03_P2.54mm_Vertical, F.Cu at (79.1, 58.4)
- added R-SW1: 10K, Resistor_SMD:R_0805_2012Metric_Pad1.20x1.40mm_HandSolder, B.Cu at (73.3, 42.7)
- added R-SW2: 10K, Resistor_SMD:R_0805_2012Metric_Pad1.20x1.40mm_HandSolder, B.Cu at (73.3, 40.6)
- added R-SW3: 10K, Resistor_SMD:R_0805_2012Metric_Pad1.20x1.40mm_HandSolder, B.Cu at (73.4, 44.8)
- added SW-PAGE1: SW_Push, Button_Switch_THT:SW_PUSH_6mm, F.Cu at (67.3, 33.7)
- added SW-SEND1: SW_Push, Button_Switch_THT:SW_PUSH_6mm, F.Cu at (67.4, 50.0)
- added SW-WIFI1: SW_Push, Button_Switch_THT:SW_PUSH_6mm, F.Cu at (67.4, 41.9)
- R-PROG1, R-PROG2, R-PROG3, R-PROG4, R-PROG5: moved to B.Cu
- moved R-PROG3 194.6 mm to (73.2, 34.8), turned to 180 degrees
- moved J-PROG1 192.5 mm to (74.1, 52.8), turned to 90 degrees
- moved R-PROG4 182.3 mm to (73.2, 32.7), turned to 180 degrees
- moved R-PROG2 177.4 mm to (86.3, 42.6)
- moved R-PROG5 174.5 mm to (86.3, 44.7)
- moved R-PROG1 172.5 mm to (86.3, 40.6)
- moved U1 164.1 mm to (79.8, 36.2)
- moved Brd1 115.4 mm to (102.5, 37.3), turned to 90 degrees
Connections:
- U1 pad 5: Net-(U1-Pad5) -> /BTN_PAGE
- U1 pad 6: Net-(U1-Pad6) -> /BTN_WIFI
- U1 pad 7: Net-(U1-Pad7) -> /BTN_SEND
Routing:
- net GND: track 0.00 -> 95.3 mm, vias 0 -> 6
- net VDD: track 0.00 -> 72.4 mm, vias 0 -> 3
- net /TX: track 0.00 -> 34.2 mm, vias 0 -> 3
- net /RST: track 0.00 -> 31.4 mm, vias 0 -> 2
- net /RX: track 0.00 -> 28.2 mm, vias 0 -> 1
- net /BTN_PAGE: track 0.00 -> 23.5 mm, vias 0 -> 2
- net /P0: track 0.00 -> 23.4 mm, vias 0 -> 2
- net /BTN_SEND: track 0.00 -> 21.4 mm, vias 0 -> 2
- net /BTN_WIFI: track 0.00 -> 17.2 mm, vias 0 -> 2
- net /LCD_SDA: track 0.00 -> 13.3 mm, vias 0 -> 1
- net /LCD_SCL: track 0.00 -> 10.5 mm, vias 0 -> 1
- net /EN: track 0.00 -> 7.23 mm, vias 0 -> 1
- net /P2: track 0.00 -> 6.02 mm, vias 0 -> 1
- net /P15: track 0.00 -> 5.27 mm, vias 0 -> 1
- added copper zone on B.Cu, net (none)
- added copper zone on F.Cu, net (none)
Other:
- board outline added: 35.9 x 34.3 mm
