File: prototrial/circuit/esp32lcd/esp32lcd.sch (KiCad schematic (older format))
At the start: 16 parts, among them SW1 SW_Push, SW2 SW_Push, SW3 SW_Push, U1 ESP32-WROOM-32

Commit message: Mic result seems weird
Parts:
- added D-RUN1: LED, symbol Device:LED
- added R-LED1: 330, symbol Device:R
Connections:
- net labels added: LED
- wire segments 59 -> 63
Changed lines of the file:
@@
 Text Label 6950 4550 0    50   ~ 0
 ESP_FLASH
+Wire Wire Line
+	5150 2450 5350 2450
+Text Label 5350 2450 0    50   ~ 0
+LED
+$Comp
+L Device:R R-LED1
+U 1 1 620BB146
+P 8150 4400
+F 0 "R-LED1" H 8220 4446 50  0001 L CNN
+F 1 "330" H 8220 4400 50  0000 L CNN
+F 2 "" V 8080 4400 50  0001 C CNN
+F 3 "~" H 8150 4400 50  0001 C CNN
+	1    8150 4400
+	1    0    0    -1
+$EndComp
+$Comp
+L power:VDD #PWR020
+U 1 1 620BB813
+P 8150 4150
+F 0 "#PWR020" H 8150 4000 50  0001 C CNN
+F 1 "VDD" H 8165 4323 50  0000 C CNN
+F 2 "" H 8150 4150 50  0001 C CNN
+F 3 "" H 8150 4150 50  0001 C CNN
+	1    8150 4150
+	1    0    0    -1
+$EndComp
+$Comp
+L Device:LED D-RUN1
+U 1 1 620BBD14
+P 8150 4800
+F 0 "D-RUN1" V 8189 4682 50  0001 R CNN
+F 1 "LED" V 8143 4682 50  0001 R CNN
+F 2 "" H 8150 4800 50  0001 C CNN
+F 3 "~" H 8150 4800 50  0001 C CNN
+	1    8150 4800
+	0    -1   -1   0
+$EndComp
+Wire Wire Line
+	8150 4550 8150 4650
+Wire Wire Line
+	8150 4150 8150 4250
+Wire Wire Line
+	8150 4950 8150 5100
+Text Label 8150 5100 0    50   ~ 0
+LED
 $EndSCHEMATC

Commit message: try re-drafting to Altium
Parts:
- added R-OLED1, R-OLED2: 10K, symbol Device:R
Connections:
- wire segments 63 -> 69
Changed lines of the file:
@@
 	1    0    0    -1
 $EndComp
-Wire Wire Line
-	7050 3450 7200 3450
-Wire Wire Line
-	7050 3350 7200 3350
-Text Label 7200 3350 0    50   ~ 0
+Text Label 7300 3350 0    50   ~ 0
 OLED_SDA
-Text Label 7200 3450 0    50   ~ 0
+Text Label 7300 3450 0    50   ~ 0
 OLED_SDL
 $Comp
@@
 Text Label 8150 5100 0    50   ~ 0
 LED
+$Comp
+L Device:R R-OLED1
+U 1 1 621610CD
+P 7100 3100
+F 0 "R-OLED1" H 7170 3146 50  0000 L CNN
+F 1 "10K" H 7170 3055 50  0000 L CNN
+F 2 "" V 7030 3100 50  0001 C CNN
+F 3 "~" H 7100 3100 50  0001 C CNN
+	1    7100 3100
+	1    0    0    -1
+$EndComp
+Wire Wire Line
+	7050 3450 7100 3450
+Wire Wire Line
+	7050 3350 7200 3350
+$Comp
+L Device:R R-OLED2
+U 1 1 6216714C
+P 7200 3100
+F 0 "R-OLED2" H 7270 3146 50  0000 L CNN
+F 1 "10K" H 7270 3055 50  0000 L CNN
+F 2 "" V 7130 3100 50  0001 C CNN
+F 3 "~" H 7200 3100 50  0001 C CNN
+	1    7200 3100
+	1    0    0    -1
+$EndComp
+Wire Wire Line
+	7200 3250 7200 3350
+Connection ~ 7200 3350
+Wire Wire Line
+	7200 3350 7300 3350
+Wire Wire Line
+	7100 3250 7100 3450
+Connection ~ 7100 3450
+Wire Wire Line
+	7100 3450 7300 3450
+$Comp
+L power:VDD #PWR021
+U 1 1 6216A0BA
+P 7150 2950
+F 0 "#PWR021" H 7150 2800 50  0001 C CNN
+F 1 "VDD" H 7165 3123 50  0000 C CNN
+F 2 "" H 7150 2950 50  0001 C CNN
+F 3 "" H 7150 2950 50  0001 C CNN
+	1    7150 2950
+	1    0    0    -1
+$EndComp
+Wire Wire Line
+	7200 2950 7150 2950
+Wire Wire Line
+	7100 2950 7150 2950
+Connection ~ 7150 2950
 $EndSCHEMATC
