File: actual/circuit/skema_p3/skema_p3.kicad_sch (KiCad schematic)
At the start: 0 parts

Commit message: P3 in KiCAD
Other:
- added sheet power (power.kicad_sch)
- sheet audio ports: added 4V6_DAC; removed 3V3_DAC, 4V6
- sheet esp32 ports: added none; removed 3V3_OLED
