File: actual/circuit/skema_p3/esp32.kicad_sch (KiCad schematic)
At the start: 10 parts, among them U1 ESP32-WROOM-32

Commit message: P3 in KiCAD Schematic
Parts:
- added J1: Conn_01x04_Male, symbol Connector:Conn_01x04_Male
Connections:
- net ESP_VDD: now also J1.1 (Pin_1)
- net GND: now also J1.4 (Pin_4)
- net RX0: now also J1.2 (Pin_2)
- net TX0: now also J1.3 (Pin_3)
Other:
- note added: "ESP32 Subsystem"
- moved on the sheet: C1, R1, R2, R3, R4, R5, R6, R7, R8, U1

Commit message: P3 in KiCAD
Parts:
- added Brd1: SSD1306, symbol SSD1306-128x64_OLED:SSD1306
- added C2, C3, C4, C7: 4.7uF, symbol Device:C
- added C5, C6: 22pF, symbol Device:C
- added R10, R11, R12, R13, R9: 10K, symbol Device:R
- added R14, R15: 1K, symbol Device:R
- added R16: 0, symbol Device:R
- added SW1, SW2, SW3, SW4, SW5: SW_Push, symbol Switch:SW_Push
Connections:
- net 3V3_ESP: now also R16.2
- net BTN_ACT_A: now also C2.1, R9.2, SW1.2
- net BTN_ACT_B: now also C3.1, R10.2, SW2.2
- net BTN_PAGE: now also C4.1, R11.2, SW3.2
- net ESP_NRST: now also C5.1, R12.2, SW4.2
- net ESP_VDD: now also R10.1, R11.1, R12.1, R13.1, R14.1, R15.1, R9.1
- net GND: now also Brd1.1 (GND), C2.2, C3.2, C4.2, C5.2, C6.2, C7.2, SW1.1, SW2.1, SW3.1, SW4.1, SW5.1
- net OLED_SCL: now also Brd1.3 (SCL), R14.2
- net OLED_SDA: now also Brd1.4 (SDA), R15.2
- net ESP_FLASH: now reaches U1.25 (IO0)
- net ESP_FLASH: now also C6.1, R13.2, SW5.2
- new net 3V3_OLED: Brd1.2 (VCC), C7.1, R16.1
Other:
- note added: "Buttons"
- note added: "OLED 128x64"

Commit message: P3 in KiCAD
Parts:
- added C10: 22pF, symbol Device:C
- added C8: 4.7uF, symbol Device:C
- added C9: 100nF, symbol Device:C
- added U2: INMP441, symbol INMP441:INMP441
Connections:
- net ESP_VDD: now also C10.1, C8.1, C9.1, U2.2 (VDD)
- net GND: now also C10.2, C8.2, C9.2, U2.1 (GND), U2.6 (LRC)
- net MIC_DATA: now also U2.3 (DATA)
- net MIC_SCK: now also U2.4 (BCLK)
- net MIC_WS: now also U2.5 (WS)
Other:
- note added: "INMP441 MIC"
- title: (none) -> Audiometry ESP32 User Interface
- moved on the sheet: Brd1, C1, C2, C3, C4, C5, C6, C7, J1, R1, R10, R11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

Commit message: P3 in KiCAD
Connections:
- net ADC_VBAT renamed ADC_BAT
Changed lines of the file:
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@@
-    )
-  )
-  (global_label "ADC_VBAT" (shape input) (at 64.77 100.33 0) (fields_autoplaced)
-    (effects (font (size 1.27 1.27)) (justify left))
-    (property "Intersheet References" "${INTERSHEET_REFS}" (id 0) (at 76.1941 100.2506 0)
-      (effects (font (size 1.27 1.27)) (justify left) hide)
     )
   )
@@
     )
   )
-  (global_label "STT_BAT" (shape input) (at 64.77 74.93 0) (fields_autoplaced)
-    (effects (font (size 1.27 1.27)) (justify left))
-    (property "Intersheet References" "${INTERSHEET_REFS}" (id 0) (at 74.6217 74.8506 0)
-      (effects (font (size 1.27 1.27)) (justify left) hide)
-    )
-  )
   (global_label "MIC_WS" (shape input) (at 64.77 62.23 0) (fields_autoplaced)
     (effects (font (size 1.27 1.27)) (justify left))
@@
     )
   )
-  (global_label "STT_MISC" (shape input) (at 64.77 54.61 0) (fields_autoplaced)
-    (effects (font (size 1.27 1.27)) (justify left))
-    (property "Intersheet References" "${INTERSHEET_REFS}" (id 0) (at 75.8312 54.5306 0)
-      (effects (font (size 1.27 1.27)) (justify left) hide)
-    )
-  )
   (global_label "ESP_VDD" (shape input) (at 153.67 67.31 90) (fields_autoplaced)
     (effects (font (size 1.27 1.27)) (justify left))
@@
     )
   )
-  (global_label "STT_RDY" (shape input) (at 64.77 97.79 0) (fields_autoplaced)
-    (effects (font (size 1.27 1.27)) (justify left))
-    (property "Intersheet References" "${INTERSHEET_REFS}" (id 0) (at 74.9241 97.7106 0)
-      (effects (font (size 1.27 1.27)) (justify left) hide)
-    )
-  )
   (global_label "RX_ESP" (shape input) (at 64.77 69.85 0) (fields_autoplaced)
     (effects (font (size 1.27 1.27)) (justify left))
@@
     )
   )
-  (global_label "STT_RUN" (shape input) (at 64.77 77.47 0) (fields_autoplaced)
-    (effects (font (size 1.27 1.27)) (justify left))
-    (property "Intersheet References" "${INTERSHEET_REFS}" (id 0) (at 75.2264 77.3906 0)
-      (effects (font (size 1.27 1.27)) (justify left) hide)
-    )
-  )
-  (global_label "STT_PAN" (shape input) (at 64.77 95.25 0) (fields_autoplaced)
-    (effects (font (size 1.27 1.27)) (justify left))
-    (property "Intersheet References" "${INTERSHEET_REFS}" (id 0) (at 74.9845 95.1706 0)
-      (effects (font (size 1.27 1.27)) (justify left) hide)
-    )
-  )
   (global_label "TX0" (shape input) (at 93.98 82.55 180) (fields_autoplaced)
     (effects (font (size 1.27 1.27)) (justify right))
@@
     (effects (font (size 1.27 1.27)) (justify left))
   )
+  (hierarchical_label "STT_RDY" (shape input) (at 64.77 97.79 0)
+    (effects (font (size 1.27 1.27)) (justify left))
+  )
+  (hierarchical_label "STT_PAN" (shape input) (at 64.77 95.25 0)
+    (effects (font (size 1.27 1.27)) (justify left))
+  )
+  (hierarchical_label "STT_BAT" (shape input) (at 64.77 74.93 0)
+    (effects (font (size 1.27 1.27)) (justify left))
+  )
   (hierarchical_label "3V3_ESP" (shape input) (at 95.25 30.48 0)
     (effects (font (size 1.27 1.27)) (justify left))
   )
+  (hierarchical_label "STT_MISC" (shape input) (at 64.77 54.61 0)
+    (effects (font (size 1.27 1.27)) (justify left))
+  )
+  (hierarchical_label "ADC_BAT" (shape input) (at 64.77 100.33 0)
+    (effects (font (size 1.27 1.27)) (justify left))
+  )
   (hierarchical_label "3V3_OLED" (shape input) (at 246.38 30.48 0)
     (effects (font (size 1.27 1.27)) (justify left))
@@
     (effects (font (size 1.27 1.27)) (justify left))
   )
+  (hierarchical_label "STT_RUN" (shape input) (at 64.77 77.47 0)
+    (effects (font (size 1.27 1.27)) (justify left))
+  )

Commit message: P3 in KiCAD
Other:
- moved on the sheet: Brd1, C1, C10, C2, C3, C4, C5, C6, C7, C8, C9, J1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

Commit message: P3 in KiCAD
Connections:
- net 3V3_OLED: no longer names the net of Brd1.2 (VCC), C7.1, R16.1
Changed lines of the file:
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@@
-    (stroke (width 0) (type default) (color 0 0 0 0))
-  )
-  (wire (pts (xy 255.27 69.85) (xy 246.38 69.85))
     (stroke (width 0) (type default) (color 0 0 0 0))
   )
@@
   )
   (wire (pts (xy 127 68.58) (xy 127 69.85))
-    (stroke (width 0) (type default) (color 0 0 0 0))
-  )
-  (wire (pts (xy 246.38 69.85) (xy 246.38 74.93))
     (stroke (width 0) (type default) (color 0 0 0 0))
   )
@@
     (effects (font (size 1.27 1.27) (thickness 0.254) bold) (justify left))
   )
-  (hierarchical_label "3V3_OLED" (shape input) (at 255.27 69.85 0)
-    (effects (font (size 1.27 1.27) (thickness 0.254) bold) (justify left))
-  )
