File: actual/circuit/skema_p3/stm32.kicad_sch (KiCad schematic)
At the start: 1 part

Commit message: P3 in KiCAD
Parts:
- added C11: 4.7uF, symbol Device:C
- added R17: 10K, symbol Device:R
- gave numbers to parts that had none: 1
Connections:
- net BTN_C: now reaches U3.10 (PC2)
- net MMC_DET: now reaches U3.11 (PC3)
- net LED_RUN: now reaches U3.15 (PA1)
- net LED_TRUE: now reaches U3.16 (PA2)
- net LED_FALSE: now reaches U3.17 (PA3)
- net LED_A: now reaches U3.20 (PA4)
- net ADC_BAT: now reaches U3.21 (PA5)
- net LED_B: now reaches U3.26 (PB0)
- net LED_C: now reaches U3.27 (PB1)
- net STT_MISC: now reaches U3.28 (PB2)
- net at U3.30 (PB11): now also C11.1
- net DAC_LRC: now reaches U3.33 (PB12)
- net DAC_BCLK: now reaches U3.34 (PB13)
- net DAC_DIN: now reaches U3.36 (PB15)
- net STT_RUN: now reaches U3.37 (PC6)
- net STT_BAT: now reaches U3.38 (PC7)
- net STT_RDY: now reaches U3.39 (PC8)
- net STT_PAN: now reaches U3.40 (PC9)
- net STM32_TX: now reaches U3.42 (PA9)
- net STM32_RX: now reaches U3.43 (PA10)
- net USB_DM: now reaches U3.44 (PA11)
- net USB_DP: now reaches U3.45 (PA12)
- net USB_DP: now also R17.2
- net SWD_IO: now reaches U3.46 (PA13)
- net SWD_CLK: now reaches U3.49 (PA14)
- net MMC_NSS: now reaches U3.50 (PA15)
- net MCC_SCK: now reaches U3.51 (PC10)
- net MMC_MISO: now reaches U3.52 (PC11)
- net MMC_MOSI: now reaches U3.53 (PC12)
- net AUDIO_RELAY: now reaches U3.58 (PB6)
- net GND: now reaches U3.60 (BOOT0)
- net GND: now also C11.2
- net STM_NRST: now reaches U3.7 (NRST)
- net BTN_A: now reaches U3.8 (PC0)
- net BTN_B: now reaches U3.9 (PC1)
- new net STM_VDD: R17.1
- no-connect marks 0 -> 21
Other:
- moved on the sheet: U3

Commit message: P3 in KiCAD
Parts:
- added C12, C16: 4.7uF, symbol Device:C
- added C13, C14: 100nF, symbol Device:C
- added C15: 22pF, symbol Device:C
- added D1, D2, D3: YELLOW, symbol Device:LED
- added D4: GREEN, symbol Device:LED
- added D5: RED, symbol Device:LED
- added D6: BLUE, symbol Device:LED
- added J2: Conn_01x05_Male, symbol Connector:Conn_01x05_Male
- added J3: USB_B_Micro, symbol Connector:USB_B_Micro
- added J4: Micro_SD_Card_Det_Hirose_DM3AT, symbol Connector:Micro_SD_Card_Det_Hirose_DM3AT
- added R18, R29: 0, symbol Device:R
- added R19, R20, R21, R22, R27, R28, R30, R31, R32: 10K, symbol Device:R
- added R23, R24, R25: 1K, symbol Device:R
- added R26: 68, symbol Device:R
- added SW6, SW7, SW8, SW9: SW_Push, symbol Switch:SW_Push
- R17: value 10K -> 68
Connections:
- net BTN_A: now also D1.1 (K), R19.2, SW6.2
- net BTN_B: now also D2.1 (K), R20.2, SW7.2
- net BTN_C: now also D3.1 (K), R21.2, SW8.2
- net GND: now also U3.12 (VSSA), U3.31 (VSS), U3.47 (VSS), U3.63 (VSS), C12.2, C13.2, C14.2, C15.2, C16.2, J2.3 (Pin_3), J3.5 (GND), J3.6 (Shield), J4.11 (SHIELD), J4.6 (VSS), J4.9 (DET_B), SW6.1, SW7.1, SW8.1, SW9.1
- net LED_FALSE: now also D5.1 (K)
- net LED_RUN: now also D6.1 (K)
- net LED_TRUE: now also D4.1 (K)
- net MCC_SCK: now also J4.5 (CLK)
- net MMC_DET: now also J4.10 (DET_A), R31.1
- net MMC_MISO: now also J4.7 (DAT0), R30.2
- net MMC_MOSI: now also J4.3 (CMD)
- net MMC_NSS: now also J4.2 (DAT3/CD)
- net STM_NRST: now also C15.1, J2.5 (Pin_5), R22.2, SW9.2
- net STM_VDD: now also U3.1 (VBAT), U3.13 (VDDA), U3.19 (VDD), U3.32 (VDD), U3.48 (VDD), U3.64 (VDD), C12.1, C13.1, C14.1, J2.1 (Pin_1), R18.1, R19.1, R20.1, R21.1, R22.1, R23.1, R24.1, R25.1, R27.2, R29.2; no longer R17.1
- net SWD_CLK: now also J2.2 (Pin_2)
- net SWD_IO: now also J2.4 (Pin_4)
- net USB_DM: now also R26.2
- net USB_DP: now also R27.1
- new net: D4.2 (A), D5.2 (A), R24.2
- new net: D1.2 (A), D2.2 (A), D3.2 (A), R23.2
- new net: D6.2 (A), R25.2
- new net: J3.2 (D-), R26.1
- new net: J3.3 (D+), R17.1
- new net: J4.1 (DAT2), R28.2
- new net: J4.8 (DAT1), R32.2
- new net 3V3_STM: R18.2
- new net CARD_VDD: C16.1, J4.4 (VDD), R28.1, R29.1, R30.1, R31.2, R32.1
Other:
- note added: "Connectors"
- note added: "LEDs and Buttons"
- note added: "STM32 Subsystem"
- title: (none) -> STM32 Audiometry Controller
- moved on the sheet: C11, U3

Commit message: P3 in KiCAD
Other:
- moved on the sheet: C11, C12, C13, C14, C15, C16, D1, D2, D3, D4, D5, D6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

Commit message: P3 in KiCAD
Connections:
- net BTN_A: no longer D1.1 (K)
- net BTN_B: no longer D2.1 (K)
- net BTN_C: no longer D3.1 (K)
- net LED_A: now also D1.1 (K)
- net LED_B: now also D2.1 (K)
- net LED_C: now also D3.1 (K)
- no-connect marks 21 -> 23
Changed lines of the file:
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@@
   (no_connect (at 72.39 81.28))
   (no_connect (at 72.39 139.7))
+  (no_connect (at 215.9 102.87))
   (no_connect (at 72.39 116.84))
   (no_connect (at 72.39 114.3))
@@
   (no_connect (at 72.39 121.92))
   (no_connect (at 72.39 60.96))
+  (no_connect (at 215.9 113.03))
   (wire (pts (xy 82.55 45.72) (xy 95.25 45.72))
     (stroke (width 0) (type default) (color 0 0 0 0))
@@
     )
   )
-  (global_label "BTN_A" (shape input) (at 125.73 111.76 270) (fields_autoplaced)
-    (effects (font (size 1.27 1.27)) (justify right))
-    (property "Intersheet References" "${INTERSHEET_REFS}" (id 0) (at 125.6506 119.7974 90)
+  (global_label "LED_A" (shape input) (at 125.73 111.76 270) (fields_autoplaced)
+    (effects (font (size 1.27 1.27)) (justify right))
+    (property "Intersheet References" "${INTERSHEET_REFS}" (id 0) (at 125.6506 119.6764 90)
       (effects (font (size 1.27 1.27)) (justify right) hide)
     )
@@
     )
   )
-  (global_label "BTN_B" (shape input) (at 135.89 111.76 270) (fields_autoplaced)
-    (effects (font (size 1.27 1.27)) (justify right))
-    (property "Intersheet References" "${INTERSHEET_REFS}" (id 0) (at 135.8106 119.9788 90)
+  (global_label "LED_B" (shape input) (at 135.89 111.76 270) (fields_autoplaced)
+    (effects (font (size 1.27 1.27)) (justify right))
+    (property "Intersheet References" "${INTERSHEET_REFS}" (id 0) (at 135.8106 119.8579 90)
       (effects (font (size 1.27 1.27)) (justify right) hide)
     )
@@
     )
   )
-  (global_label "BTN_C" (shape input) (at 146.05 111.76 270) (fields_autoplaced)
-    (effects (font (size 1.27 1.27)) (justify right))
-    (property "Intersheet References" "${INTERSHEET_REFS}" (id 0) (at 145.9706 119.9788 90)
-      (effects (font (size 1.27 1.27)) (justify right) hide)
-    )
+  (global_label "LED_C" (shape input) (at 146.05 111.76 270) (fields_autoplaced)
+    (effects (font (size 1.27 1.27)) (justify right))
+    (property "Intersheet References" "${INTERSHEET_REFS}" (id 0) (at 145.9706 119.8579 90)
+      (effects (font (size 1.27 1.27)) (justify right) hide)
+    )

Commit message: P3 in KiCAD
Parts:
- added J9: Conn_01x03_Male, symbol Connector:Conn_01x03_Male
Connections:
- net GND: now also J9.3 (Pin_3)
- net STM32_RX: now also J9.2 (Pin_2)
- net STM32_TX: now also J9.1 (Pin_1)
Changed lines of the file:
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@@
     (effects (font (size 1.27 1.27) (thickness 0.254) bold) (justify left))
+  )
+  (hierarchical_label "STM32_RX" (shape input) (at 106.68 86.36 180)
+    (effects (font (size 1.27 1.27) (thickness 0.254) bold) (justify right))
+  )
+  (hierarchical_label "STM32_TX" (shape input) (at 106.68 83.82 180)
+    (effects (font (size 1.27 1.27) (thickness 0.254) bold) (justify right))
   )
   (hierarchical_label "STM32_TX" (shape input) (at 72.39 83.82 0)
@@
     (pin "2")
   )
+  (symbol (lib_id "Connector:Conn_01x03_Male") (at 111.76 86.36 0) (mirror y) (unit 1)
+    (in_bom yes) (on_board yes) (fields_autoplaced)
+    (property "Reference" "J9" (id 0) (at 113.03 86.3599 0)
+      (effects (font (size 1.27 1.27)) (justify right))
+    )
+    (property "Value" "Conn_01x03_Male" (id 1) (at 113.03 87.6299 0)
+      (effects (font (size 1.27 1.27)) (justify right) hide)
+    )
+    (property "Footprint" "" (id 2) (at 111.76 86.36 0)
+      (effects (font (size 1.27 1.27)) hide)
+    )
+    (property "Datasheet" "~" (id 3) (at 111.76 86.36 0)
+      (effects (font (size 1.27 1.27)) hide)
+    )
+    (pin "1")
+    (pin "2")
+    (pin "3")
+  )
   (symbol (lib_id "Device:LED") (at 176.53 107.95 90) (unit 1)
     (in_bom yes) (on_board yes)
@@
     (pin "2")
   )
+  (symbol (lib_id "power:GND") (at 106.68 88.9 0) (unit 1)
+    (in_bom yes) (on_board yes) (fields_autoplaced)
+    (property "Reference" "#PWR057" (id 0) (at 106.68 95.25 0)
+      (effects (font (size 1.27 1.27)) hide)
+    )
+    (property "Value" "GND" (id 1) (at 106.68 93.98 0))
+    (property "Footprint" "" (id 2) (at 106.68 88.9 0)
+      (effects (font (size 1.27 1.27)) hide)
+    )
+    (property "Datasheet" "" (id 3) (at 106.68 88.9 0)
+      (effects (font (size 1.27 1.27)) hide)
+    )
+    (pin "1")
+  )
   (symbol (lib_id "Switch:SW_Push") (at 129.54 71.12 90) (unit 1)
